File: KiCad/RobotASK/Photoresistor-array/Photoresistor-array.kicad_sch (KiCad schematic)
At the start: 10 parts, among them J1 Conn_01x04_Pin, J2 Conn_01x02_Pin

Commit message: Poprawki kodu, zwiększenie otworów na komponenty na 1mm, nowe wydruki do termotransferu i nawiercania otworów, poukładanie nieaktualnych wydruków UV
Parts:
- R1, R2, R3, R4: footprint Resistor_THT:R_Axial_DIN0207_L6.3mm_D2.5mm_P10.16mm_Horizontal -> Library:R_Axial_DIN0207_L6.3mm_D2.5mm_P10.16mm_Horizontal
- R5, R6, R7, R8: footprint OptoDevice:R_LDR_5.1x4.3mm_P3.4mm_Vertical -> Library:R_LDR_5.1x4.3mm_P3.4mm_Vertical

Commit message: renders
Other:
- title: (none) -> Piano Tiles robot - photoresistor array module
- moved on the sheet: J1, J2, R1, R2, R3, R4, R5, R6, R7, R8
